File: designs/arena_10_of_10_v1r1/fan_out.kicad_sch (KiCad schematic)
At the start: 4 parts, among them U2 74LVC2G17

Commit message: Re-worked MISO handling and analog input circuit.
Modified so that MISO isolation circuits are in fan out section and
are such that they will be placed close to the teensy.  Modified the
analog input circuit so that the teensy MCU analog inputs are used in
conjuction with a level shifting circuit.
Parts:
- removed C1: 0.1uF, Capacitor_SMD:C_0402_1005Metric, symbol Device:C
- removed R? (x2): 33, symbol Device:R_Small
- removed U2: 74LVC2G17, Package_TO_SOT_SMD:SOT-23-6, symbol 74xGxx:74LVC2G17
Other:
- added sheet MISO B0 Enable for P1 (miso_enable.kicad_sch)
- added sheet MISO B0 Enable for P2 (miso_enable.kicad_sch)
- added sheet MISO B0 Enable for P3 (miso_enable.kicad_sch)
- added sheet MISO B0 Enable for P4 (miso_enable.kicad_sch)
- added sheet MISO B0 Enable for P5 (miso_enable.kicad_sch)
- added sheet MISO B1 Enable for P10 (miso_enable.kicad_sch)
- added sheet MISO B1 Enable for P6 (miso_enable.kicad_sch)
- added sheet MISO B1 Enable for P7 (miso_enable.kicad_sch)
- added sheet MISO B1 Enable for P8 (miso_enable.kicad_sch)
- added sheet MISO B1 Enable for P9 (miso_enable.kicad_sch)
- note added: "SPI Bus B0 MISO for columns P1-P5"
- note added: "SPI Bus B1 MISO for columns P6-P10"
- note added: "SPI Bus B1 MOSI for columns P6-P10"
- note removed: "MISO lines coming back to MCU. Not really fan out (1x), but needed to put them somewhere"
- note removed: "SN74LVC2G17DBVR C10429"
- note removed: "SPI Bus B0 MISO"
- note removed: "SPI Bus B1 MISO"
- note removed: "SPI Bus B1 MOSI for columns P1-P5"
