File: designs/arena_10_of_10_v1r1/panels.kicad_sch (KiCad schematic)
At the start: 0 parts

Commit message: Re-worked MISO handling and analog input circuit.
Modified so that MISO isolation circuits are in fan out section and
are such that they will be placed close to the teensy.  Modified the
analog input circuit so that the teensy MCU analog inputs are used in
conjuction with a level shifting circuit.
Other:
- note added: "SPI Bus B0 MISO for columns P1-P5"
- note added: "SPI Bus B1 MISO for columns P6-P10"
- note added: "SPI Bus B1 MOSI for columns P6-P10"
- note removed: "SPI Bus B0 MISO"
- note removed: "SPI Bus B1 MISO"
- note removed: "SPI Bus B1 MOSI for columns P1-P5"
