File: designs/arena_10_of_10_v1r1/teensy.kicad_sch (KiCad schematic)
At the start: 35 parts, among them U1 Teensy4.1

Commit message: Re-worked MISO handling and analog input circuit.
Modified so that MISO isolation circuits are in fan out section and
are such that they will be placed close to the teensy.  Modified the
analog input circuit so that the teensy MCU analog inputs are used in
conjuction with a level shifting circuit.
Connections:
- net A0 renamed AIN.A0
- net A1 renamed AIN.A1
Other:
- note added: "To do 1. Add external ethernet"
- note removed: "To do ... 1. Add -5V supply 2. Add external ethernet"
- moved on the sheet: C?, J?, U?
