File: arena_10-10/arena_top_10-10/panel_column.kicad_sch (KiCad schematic)
At the start: 4 parts, among them J5 Conn_01x05, J6 Conn_01x05, P1 NA

Commit message: Pushed latest minor changes.
Checked lscs parts numbers.  Added some images. remade production files.
Parts:
- J5, J6: LCSC Part # C50950 -> C492404
Changed lines of the file:
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@@
 			)
 		)
-		(property "LCSC Part #" "C50950"
+		(property "LCSC Part #" "C492404"
 			(at 161.29 69.85 0)
 			(effects
@@
 			)
 		)
-		(property "LCSC Part #" "C50950"
+		(property "LCSC Part #" "C492404"
 			(at 161.29 85.09 0)
 			(effects
